Commit message: Update leaf.urdf to match nrc_svcs, and av_ui.py to use nrc_av_ui's paramsForDriving.sh

File: scripts/leaf.urdf (robot description, URDF)
Before this commit: robot leaf_test, 36 links, 35 joints
Links:
- added link cubtek_L; visual box size=0.05 0.05 0.05
- added link cubtek_R; visual box size=0.05 0.05 0.05
Joints:
- added joint cubtek_L: type fixed, parent sensor_hub, child cubtek_L, origin xyz=3.53 0.73 -0.32 rpy=0 0.0 0.872665
- added joint cubtek_R: type fixed, parent sensor_hub, child cubtek_R, origin xyz=3.53 -0.742 -0.32 rpy=0 0.0 -0.872665
